File: hardware/compact.sch (EAGLE design)
At the start: 30 parts, among them IC1 ATMEGA168-20P, IC3 MAX232

Commit message: Updated hardware.
Parts:
- C12: device rcl:CPOL-EUE2.5-6 -> rcl:CPOL-EUE2.5-5
- IC1: value ATMEGA168-20P -> MEGA8-PU; device adafruit:ATMEGA168-20P -> avr-6:MEGA8-PU
- L1: device rcl:L-EU0204/7 -> rcl:L-EU0207/5V
- Q1: value (none) -> 16MHz
- R6: device rcl:R-EU_0204/2V -> rcl:R-EU_0204/5
Connections:
- removed net N$26: IC1.(PCI11/ADC3)PC3, U$2DDS-1.CLK
- removed net N$30: IC1.(PCI9/ADC1)PC1, U$2DDS-1.D7
- new net N$18: IC1.PD6(AIN0), U$2DDS-1.CLK
- new net N$19: IC1.PB0(ICP1), U$2DDS-1.D7
- net GND: now also IC1.GND@1; no longer IC1.GND
- net N$1: now also IC1.PC6(/RESET); no longer IC1.PC6(/RESET/PCI14)
- net N$15: now also IC1.PD7(AIN1); no longer IC1.(PCI10/ADC2)PC2
- net N$17: now also IC1.PD1(TXD); no longer IC1.(PCI17/TXD)PD1
- net N$22: now also IC1.PD0(RXD); no longer IC1.(PCI16/RXD)PD0
- net N$5: now also IC1.PB7(XTAL2/TOSC2); no longer IC1.PB7(XTAL2/TOSC2/PCI7)
- net N$6: now also IC1.PB6(XTAL1/TOSC1); no longer IC1.PB6(XTAL1/TOSC1/PCI6)
- net N$9: now also IC1.PC4(ADC4/SDA); no longer IC1.(PCI13/ADC5/SCL)PC5
- net VCC: now also IC1.VCC@1; no longer IC1.VCC
Other:
- moved on the sheet: C5, C7, C8, Q1, R4, R5, R6

Commit message: Fixed circuit and board.
Parts:
- C10: device rcl:CPOL-EUE5-5 -> rcl:CPOL-EUE2.5-6
- C5: device rcl:C-EU050-025X075 -> rcl:C-EU102-043X133
- JP8: value RS-232 -> RS-232 GndTxRx
- Q1: device crystal:CRYSTALHC18U-V -> crystal:CRYSTALHC49U-V
Connections:
- removed net N$13: U$1.C1B, U$2DDS-1.SIN-
- new net N$1: U$1.C2B, U$2DDS-1.SIN-
- net N$14: now also U$1.C1B; no longer U$1.C2B
Other:
- moved on the sheet: C10, C11, C12, C13, C5, C7, C8, IC1, IC3, JP8, Q1, R4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

Commit message: Fixes.
Parts:
- removed U$2: DDS-1, minikits:DDS-1
- added C14, C9: 220nF, rcl:C-EU025-025X050
- added C15: 100nF, rcl:C-EU050-025X075
- added C16: 100nF, rcl:C-EU075-032X103
- added C4: 100nF, rcl:C-EU025-025X050
- added JP2: DTR, pinhead:PINHD-1X1
- added L2: 10uH, rcl:L-EU0204/7
- added R10, R11, R9: 220, rcl:R-EU_0204/2V
- added R7: 1k, resistor:R-TRIMM74W
- added R8: 100, rcl:R-EU_0204/2V
- added T1, T2: 2N3904, transistor-neu-to92:2N3904-NPN-TO92-EBC
- C6: device rcl:C-EU050-025X075 -> rcl:C-EU025-025X050
- R2, R4: device rcl:R-EU_0204/7 -> rcl:R-EU_0204/5
- R3: device rcl:R-EU_0204/5 -> rcl:R-EU_0204/2V
- U$1: value T37_TRANSFORMER -> DDS-1; device toroid:T37_TRANSFORMER -> minikits:DDS-1
Connections:
- new net N$13: C4.1, R7.A
- new net N$20: C9.1, L2.1, R10.1, T2.C
- new net N$21: R10.2, T1.C, T2.B
- new net N$23: C15.2, JP7.1
- new net N$24: C15.1, R11.2, R9.2, T2.E
- new net N$26: C16.1, IC3G$1.R2OUT
- new net N$27: IC3G$1.R2IN, JP2.1
- net GND: now also C14.2, C9.2, R11.1, R8.2, T1.E, U$1DDS-1.D2, U$1DDS-1.RESET, U$1G$2.GND; no longer U$1.C1A, U$1.C2A, U$2DDS-1.D2, U$2DDS-1.RESET, U$2G$2.GND
- net N$1: now also C4.2, U$1DDS-1.SIN-; no longer U$1.C2B, U$2DDS-1.SIN-
- net N$14: now also R7.E, R7.S, R8.1, R9.1, T1.B; no longer JP7.1, U$1.C1B
- net N$15: now also U$1DDS-1.FQ_UD; no longer U$2DDS-1.FQ_UD
- net N$18: now also U$1DDS-1.CLK; no longer U$2DDS-1.CLK
- net N$19: now also U$1DDS-1.D7; no longer U$2DDS-1.D7
- net N$25: now also C16.2
- net VCC: now also C14.1, L2.2, U$1DDS-1.D0, U$1DDS-1.D1, U$1G$2.VCC; no longer U$2DDS-1.D0, U$2DDS-1.D1, U$2G$2.VCC
Other:
- note added: "Optional"
- note removed: "16:4T"
- moved on the sheet: C21, JP7, L1
