File: hardware/prg.sch (EAGLE design)
At the start: 3 parts, among them IC1 MEGA8-PU

Commit message: Fixes.
Parts:
- added C1: 22pF, rcl:C-EU025-025X050
- added C2: 22pF, rcl:C-EU050-025X075
- added Q1: 16MHz, crystal:CRYSTALHC49S
Connections:
- removed net N$6: IC1.PC6(/RESET), JP1.5, R1.1
- new net GND: C1.1, C2.1, IC1.GND@1, JP1.6
- new net N$7: IC1.PC6(/RESET), JP1.5, R1.2
- new net VCC: IC1.VCC@1, JP1.2, R1.1
- net N$4: now also C2.2, IC1.PB7(XTAL2/TOSC2), Q1.1; no longer IC1.GND@1, JP1.6
- net N$5: now also C1.2, IC1.PB6(XTAL1/TOSC1), Q1.2; no longer IC1.VCC@1, JP1.2, R1.2
Other:
- moved on the sheet: R1
Changed lines of the file:
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@@
 <part name="JP1" library="avr-6" deviceset="AVR-ISP-6" device=""/>
 <part name="R1" library="rcl" deviceset="R-EU_" device="0204/7" value="10k"/>
+<part name="Q1" library="crystal" deviceset="CRYSTAL" device="HC49S" value="16MHz"/>
+<part name="C1" library="rcl" deviceset="C-EU" device="025-025X050" value="22pF"/>
+<part name="C2" library="rcl" deviceset="C-EU" device="050-025X075" value="22pF"/>
+<part name="GND1" library="supply1" deviceset="GND" device=""/>
+<part name="GND2" library="supply1" deviceset="GND" device=""/>
+<part name="GND3" library="supply1" deviceset="GND" device=""/>
+<part name="GND4" library="supply1" deviceset="GND" device=""/>
+<part name="P+1" library="supply1" deviceset="VCC" device=""/>
+<part name="P+2" library="supply1" deviceset="VCC" device=""/>
+<part name="P+3" library="supply1" deviceset="VCC" device=""/>
 </parts>
 <sheets>
@@
 <instance part="IC1" gate="1" x="50.8" y="53.34"/>
 <instance part="JP1" gate="G$1" x="53.34" y="7.62"/>
-<instance part="R1" gate="G$1" x="12.7" y="66.04" rot="R270"/>
+<instance part="R1" gate="G$1" x="17.78" y="88.9" rot="R270"/>
+<instance part="Q1" gate="G$1" x="17.78" y="63.5" rot="R90"/>
+<instance part="C1" gate="G$1" x="10.16" y="66.04" rot="R90"/>
+<instance part="C2" gate="G$1" x="10.16" y="60.96" rot="R90"/>
+<instance part="GND1" gate="1" x="0" y="55.88"/>
+<instance part="GND2" gate="1" x="5.08" y="55.88"/>
+<instance part="GND3" gate="1" x="15.24" y="20.32"/>
+<instance part="GND4" gate="1" x="43.18" y="0"/>
+<instance part="P+1" gate="VCC" x="17.78" y="96.52"/>
+<instance part="P+2" gate="VCC" x="40.64" y="17.78"/>
+<instance part="P+3" gate="VCC" x="17.78" y="58.42"/>
 </instances>
 <busses>
@@
 <net name="N$4" class="0">
 <segment>
-<pinref part="JP1" gate="G$1" pin="6"/>
-<wire x1="48.26" y1="5.08" x2="15.24" y2="5.08" width="0.1524" layer="91"/>
-<wire x1="15.24" y1="5.08" x2="15.24" y2="25.4" width="0.1524" layer="91"/>
-<pinref part="IC1" gate="1" pin="GND@1"/>
-<wire x1="15.24" y1="25.4" x2="20.32" y2="25.4" width="0.1524" layer="91"/>
+<pinref part="IC1" gate="1" pin="PB7(XTAL2/TOSC2)"/>
+<pinref part="Q1" gate="G$1" pin="1"/>
+<wire x1="20.32" y1="60.96" x2="17.78" y2="60.96" width="0.1524" layer="91"/>
+<pinref part="C2" gate="G$1" pin="2"/>
+<wire x1="17.78" y1="60.96" x2="15.24" y2="60.96" width="0.1524" layer="91"/>
+<junction x="17.78" y="60.96"/>
 </segment>
 </net>
 <net name="N$5" class="0">
 <segment>
-<pinref part="JP1" gate="G$1" pin="2"/>
-<wire x1="48.26" y1="10.16" x2="12.7" y2="10.16" width="0.1524" layer="91"/>
-<wire x1="12.7" y1="10.16" x2="12.7" y2="53.34" width="0.1524" layer="91"/>
-<pinref part="IC1" gate="1" pin="VCC@1"/>
-<wire x1="12.7" y1="53.34" x2="20.32" y2="53.34" width="0.1524" layer="91"/>
-<pinref part="R1" gate="G$1" pin="2"/>
-<wire x1="12.7" y1="60.96" x2="12.7" y2="53.34" width="0.1524" layer="91"/>
-<junction x="12.7" y="53.34"/>
+<pinref part="IC1" gate="1" pin="PB6(XTAL1/TOSC1)"/>
+<pinref part="Q1" gate="G$1" pin="2"/>
+<wire x1="20.32" y1="66.04" x2="17.78" y2="66.04" width="0.1524" layer="91"/>
+<pinref part="C1" gate="G$1" pin="2"/>
+<wire x1="17.78" y1="66.04" x2="15.24" y2="66.04" width="0.1524" layer="91"/>
+<junction x="17.78" y="66.04"/>
 </segment>
 </net>
-<net name="N$6" class="0">
+<net name="GND" class="0">
+<segment>
+<pinref part="C2" gate="G$1" pin="1"/>
+<pinref part="GND2" gate="1" pin="GND"/>
+<wire x1="7.62" y1="60.96" x2="5.08" y2="60.96" width="0.1524" layer="91"/>
+<wire x1="5.08" y1="60.96" x2="5.08" y2="58.42" width="0.1524" layer="91"/>
+</segment>
+<segment>
+<pinref part="C1" gate="G$1" pin="1"/>
+<pinref part="GND1" gate="1" pin="GND"/>
+<wire x1="7.62" y1="66.04" x2="0" y2="66.04" width="0.1524" layer="91"/>
+<wire x1="0" y1="66.04" x2="0" y2="58.42" width="0.1524" layer="91"/>
+</segment>
+<segment>
+<pinref part="IC1" gate="1" pin="GND@1"/>
+<pinref part="GND3" gate="1" pin="GND"/>
+<wire x1="20.32" y1="25.4" x2="15.24" y2="25.4" width="0.1524" layer="91"/>
+<wire x1="15.24" y1="25.4" x2="15.24" y2="22.86" width="0.1524" layer="91"/>
+</segment>
+<segment>
+<pinref part="JP1" gate="G$1" pin="6"/>
+<pinref part="GND4" gate="1" pin="GND"/>
+<wire x1="48.26" y1="5.08" x2="43.18" y2="5.08" width="0.1524" layer="91"/>
+<wire x1="43.18" y1="5.08" x2="43.18" y2="2.54" width="0.1524" layer="91"/>
+</segment>
+</net>
+<net name="N$7" class="0">
 <segment>
 <pinref part="IC1" gate="1" pin="PC6(/RESET)"/>
-<pinref part="R1" gate="G$1" pin="1"/>
-<wire x1="20.32" y1="81.28" x2="12.7" y2="81.28" width="0.1524" layer="91"/>
-<wire x1="12.7" y1="81.28" x2="12.7" y2="71.12" width="0.1524" layer="91"/>
+<pinref part="R1" gate="G$1" pin="2"/>
+<wire x1="20.32" y1="81.28" x2="17.78" y2="81.28" width="0.1524" layer="91"/>
+<wire x1="17.78" y1="81.28" x2="17.78" y2="83.82" width="0.1524" layer="91"/>
 <pinref part="JP1" gate="G$1" pin="5"/>
-<wire x1="48.26" y1="7.62" x2="7.62" y2="7.62" width="0.1524" layer="91"/>
-<wire x1="7.62" y1="7.62" x2="7.62" y2="81.28" width="0.1524" layer="91"/>
-<wire x1="7.62" y1="81.28" x2="12.7" y2="81.28" width="0.1524" layer="91"/>
-<junction x="12.7" y="81.28"/>
+<wire x1="48.26" y1="7.62" x2="-5.08" y2="7.62" width="0.1524" layer="91"/>
+<wire x1="-5.08" y1="7.62" x2="-5.08" y2="81.28" width="0.1524" layer="91"/>
+<wire x1="-5.08" y1="81.28" x2="17.78" y2="81.28" width="0.1524" layer="91"/>
+<junction x="17.78" y="81.28"/>
 </segment>
 </net>
+<net name="VCC" class="0">
+<segment>
+<pinref part="JP1" gate="G$1" pin="2"/>
+<pinref part="P+2" gate="VCC" pin="VCC"/>
+<wire x1="48.26" y1="10.16" x2="40.64" y2="10.16" width="0.1524" layer="91"/>
+<wire x1="40.64" y1="10.16" x2="40.64" y2="15.24" width="0.1524" layer="91"/>
+</segment>
+<segment>
+<pinref part="R1" gate="G$1" pin="1"/>
+<pinref part="P+1" gate="VCC" pin="VCC"/>
+</segment>
+<segment>
+<pinref part="IC1" gate="1" pin="VCC@1"/>
+<pinref part="P+3" gate="VCC" pin="VCC"/>
+<wire x1="20.32" y1="53.34" x2="17.78" y2="53.34" width="0.1524" layer="91"/>
+<wire x1="17.78" y1="53.34" x2="17.78" y2="55.88" width="0.1524" layer="91"/>
+</segment>
+</net>
